Commit message: complete the visual model of wukong

File: src/wukong/urdf/wukong.urdf (robot description, URDF)
Before this commit: robot WuKong, 8 links, 7 joints
Links:
- link LowerArm1: geometry visual mesh filename=package://wukong/meshes/LowerArm1.STL
- link LowerArm2: geometry visual mesh filename=package://wukong/meshes/LowerArm2.STL
- link LowerArm3: geometry visual mesh filename=package://wukong/meshes/LowerArm3.STL
- link Racket: geometry visual mesh filename=package://wukong/meshes/Racket.STL
- link Shoulder: geometry visual mesh filename=package://wukong/meshes/Shoulder.STL
- link UpperArm1: geometry visual mesh filename=package://wukong/meshes/UpperArm1.STL
- link UpperArm2: geometry visual mesh filename=package://wukong/meshes/UpperArm2.STL
- link body: geometry visual box size=0.2 0.3 0.8
Joints:
- joint ElbowRoll: origin xyz=0 0 -0.241 -> xyz=0 0 -0.221
- joint ElbowYaw: origin xyz=0 0 -0.01 -> xyz=0 0 -0.0606
- joint ShoulderRoll: origin xyz=0 -0.114 0 -> xyz=0 -0.13395 0
- joint ShoulderYaw: origin xyz=0 0 -0.02 -> xyz=0 0 -0.035
- joint WristPitch: origin xyz=0 0 -0.1 -> xyz=0 0 0
- joint WristRoll: origin xyz=0 0 -0.250 -> xyz=0 0 -0.19908

Commit message: change the appearance and color of wukong

File: src/wukong/urdf/wukong.urdf (robot description, URDF)
Before this commit: robot WuKong, 8 links, 7 joints
Joints:
- joint ElbowRoll: origin xyz=0 0 -0.221 -> xyz=0 0 -0.183
- joint ElbowYaw: origin xyz=0 0 -0.0606 -> xyz=0 0 -0.086
- joint ShoulderYaw: origin xyz=0 0 -0.035 -> xyz=0 0 -0.076
- joint WristRoll: origin xyz=0 0 -0.19908 -> xyz=0 0 -0.173
